Commit message: Minor updates to jvrc1 urdf (not loading in Pinocchio)

File: jvrc_description/jvrc1.urdf (robot description, URDF)
Before this commit: robot jvrc1, 60 links, 59 joints
Links:
- link L_ANKLE_P_S: geometry collision mesh filename=meshes/L_ANKLE_P_S.dae; visual mesh filename=meshes/L_ANKLE_P_S.dae
- link L_ELBOW_P_S: geometry collision mesh filename=meshes/L_ELBOW_P_S.dae; visual mesh filename=meshes/L_ELBOW_P_S.dae
- link L_ELBOW_Y_S: geometry collision mesh filename=meshes/L_ELBOW_Y_S.dae; visual mesh filename=meshes/L_ELBOW_Y_S.dae
- link L_HIP_R_S: geometry collision mesh filename=meshes/L_HIP_R_S.dae; visual mesh filename=meshes/L_HIP_R_S.dae
- link L_HIP_Y_S: geometry collision mesh filename=meshes/L_HIP_Y_S.dae; visual mesh filename=meshes/L_HIP_Y_S.dae
- link L_KNEE_S: geometry collision mesh filename=meshes/L_KNEE_S.dae; visual mesh filename=meshes/L_KNEE_S.dae
- link L_LINDEX_S: geometry collision mesh filename=meshes/L_LINDEX_S.dae; visual mesh filename=meshes/L_LINDEX_S.dae
- link L_LLITTLE_S: geometry collision mesh filename=meshes/L_LLITTLE_S.dae; visual mesh filename=meshes/L_LLITTLE_S.dae
- link L_LTHUMB_S: geometry collision mesh filename=meshes/L_LTHUMB_S.dae; visual mesh filename=meshes/L_LTHUMB_S.dae
- link L_SHOULDER_P_S: geometry collision mesh filename=meshes/L_SHOULDER_P_S.dae; visual mesh filename=meshes/L_SHOULDER_P_S.dae
- link L_SHOULDER_Y_S: geometry collision mesh filename=meshes/L_SHOULDER_Y_S.dae; visual mesh filename=meshes/L_SHOULDER_Y_S.dae
- link L_UINDEX_S: geometry collision mesh filename=meshes/L_UINDEX_S.dae; visual mesh filename=meshes/L_UINDEX_S.dae
- link L_ULITTLE_S: geometry collision mesh filename=meshes/L_ULITTLE_S.dae; visual mesh filename=meshes/L_ULITTLE_S.dae
- link L_UTHUMB_S: geometry collision mesh filename=meshes/L_UTHUMB_S.dae; visual mesh filename=meshes/L_UTHUMB_S.dae
- link L_WRIST_Y_S: geometry collision mesh filename=meshes/L_WRIST_Y_S.dae; visual mesh filename=meshes/L_WRIST_Y_S.dae
- link NECK_P_S: geometry collision mesh filename=meshes/NECK_P_S.dae; visual mesh filename=meshes/NECK_P_S.dae
- link NECK_Y_S: geometry collision mesh filename=meshes/NECK_Y_S.dae; visual mesh filename=meshes/NECK_Y_S.dae
- link PELVIS_S: geometry collision mesh filename=meshes/PELVIS_S.dae; visual mesh filename=meshes/PELVIS_S.dae
- link R_ANKLE_P_S: geometry collision mesh filename=meshes/R_ANKLE_P_S.dae; visual mesh filename=meshes/R_ANKLE_P_S.dae
- link R_ELBOW_P_S: geometry collision mesh filename=meshes/R_ELBOW_P_S.dae; visual mesh filename=meshes/R_ELBOW_P_S.dae
- link R_ELBOW_Y_S: geometry collision mesh filename=meshes/R_ELBOW_Y_S.dae; visual mesh filename=meshes/R_ELBOW_Y_S.dae
- link R_HIP_R_S: geometry collision mesh filename=meshes/R_HIP_R_S.dae; visual mesh filename=meshes/R_HIP_R_S.dae
- link R_HIP_Y_S: geometry collision mesh filename=meshes/R_HIP_Y_S.dae; visual mesh filename=meshes/R_HIP_Y_S.dae
- link R_KNEE_S: geometry collision mesh filename=meshes/R_KNEE_S.dae; visual mesh filename=meshes/R_KNEE_S.dae
- link R_LINDEX_S: geometry collision mesh filename=meshes/R_LINDEX_S.dae; visual mesh filename=meshes/R_LINDEX_S.dae
- link R_LLITTLE_S: geometry collision mesh filename=meshes/R_LLITTLE_S.dae; visual mesh filename=meshes/R_LLITTLE_S.dae
- link R_LTHUMB_S: geometry collision mesh filename=meshes/R_LTHUMB_S.dae; visual mesh filename=meshes/R_LTHUMB_S.dae
- link R_SHOULDER_P_S: geometry collision mesh filename=meshes/R_SHOULDER_P_S.dae; visual mesh filename=meshes/R_SHOULDER_P_S.dae
- link R_SHOULDER_Y_S: geometry collision mesh filename=meshes/R_SHOULDER_Y_S.dae; visual mesh filename=meshes/R_SHOULDER_Y_S.dae
- link R_UINDEX_S: geometry collision mesh filename=meshes/R_UINDEX_S.dae; visual mesh filename=meshes/R_UINDEX_S.dae
- link R_ULITTLE_S: geometry collision mesh filename=meshes/R_ULITTLE_S.dae; visual mesh filename=meshes/R_ULITTLE_S.dae
- link R_UTHUMB_S: geometry collision mesh filename=meshes/R_UTHUMB_S.dae; visual mesh filename=meshes/R_UTHUMB_S.dae
- link R_WRIST_Y_S: geometry collision mesh filename=meshes/R_WRIST_Y_S.dae; visual mesh filename=meshes/R_WRIST_Y_S.dae
- link WAIST_R_S: geometry collision mesh filename=meshes/WAIST_R_S.dae; visual mesh filename=meshes/WAIST_R_S.dae
- link WAIST_Y_S: geometry collision mesh filename=meshes/WAIST_Y_S.dae; visual mesh filename=meshes/WAIST_Y_S.dae
