Commit message: Feet link created

File: jvrc_description/unitreeg1.urdf (robot description, URDF)
Before this commit: robot unitreeg1, 39 links, 38 joints
Links:
- added link left_foot_link, mass 0.00001; collision sphere radius=0.005; collision sphere radius=0.005
- added link right_foot_link, mass 0.00001; collision sphere radius=0.005; collision sphere radius=0.005
Joints:
- added joint left_foot_joint: type fixed, parent left_ankle_roll_link, child left_foot_link, origin xyz=0.035 0 -0.03 rpy=0 0 0, axis 1 0 0, limit lower=-0.2618 upper=0.2618 effort=35 velocity=30
- added joint right_foot_joint: type fixed, parent right_ankle_roll_link, child right_foot_link, origin xyz=0.035 0 -0.03 rpy=0 0 0, axis 1 0 0, limit lower=-0.2618 upper=0.2618 effort=35 velocity=30

Commit message: Finally the robot walks, fixed foot lenght and removed pelvis task in order to achieve walking, remove stopping phase in order to achieve standing after walking phase, modified plots

File: jvrc_description/unitreeg1.urdf (robot description, URDF)
Before this commit: robot unitreeg1, 41 links, 40 joints
Links:
- link left_ankle_roll_link: geometry visual mesh filename=meshes/left_ankle_roll_link.STL
- link right_ankle_roll_link: geometry visual mesh filename=meshes/right_ankle_roll_link.STL
