Commit message: Minor updates to urdf structure

File: jvrc_description/urdf/jvrc1.urdf (robot description, URDF)
Before this commit: robot jvrc1, 60 links, 59 joints
Links:
- link L_ANKLE_P_S: geometry collision mesh filename=package://jvrc_description/meshes/L_ANKLE_P_S.dae; visual mesh filename=package://jvrc_description/meshes/L_ANKLE_P_S.dae
- link L_ELBOW_P_S: geometry collision mesh filename=package://jvrc_description/meshes/L_ELBOW_P_S.dae; visual mesh filename=package://jvrc_description/meshes/L_ELBOW_P_S.dae
- link L_ELBOW_Y_S: geometry collision mesh filename=package://jvrc_description/meshes/L_ELBOW_Y_S.dae; visual mesh filename=package://jvrc_description/meshes/L_ELBOW_Y_S.dae
- link L_HIP_R_S: geometry collision mesh filename=package://jvrc_description/meshes/L_HIP_R_S.dae; visual mesh filename=package://jvrc_description/meshes/L_HIP_R_S.dae
- link L_HIP_Y_S: geometry collision mesh filename=package://jvrc_description/meshes/L_HIP_Y_S.dae; visual mesh filename=package://jvrc_description/meshes/L_HIP_Y_S.dae
- link L_KNEE_S: geometry collision mesh filename=package://jvrc_description/meshes/L_KNEE_S.dae; visual mesh filename=package://jvrc_description/meshes/L_KNEE_S.dae
- link L_LINDEX_S: geometry collision mesh filename=package://jvrc_description/meshes/L_LINDEX_S.dae; visual mesh filename=package://jvrc_description/meshes/L_LINDEX_S.dae
- link L_LLITTLE_S: geometry collision mesh filename=package://jvrc_description/meshes/L_LLITTLE_S.dae; visual mesh filename=package://jvrc_description/meshes/L_LLITTLE_S.dae
- link L_LTHUMB_S: geometry collision mesh filename=package://jvrc_description/meshes/L_LTHUMB_S.dae; visual mesh filename=package://jvrc_description/meshes/L_LTHUMB_S.dae
- link L_SHOULDER_P_S: geometry collision mesh filename=package://jvrc_description/meshes/L_SHOULDER_P_S.dae; visual mesh filename=package://jvrc_description/meshes/L_SHOULDER_P_S.dae
- link L_SHOULDER_Y_S: geometry collision mesh filename=package://jvrc_description/meshes/L_SHOULDER_Y_S.dae; visual mesh filename=package://jvrc_description/meshes/L_SHOULDER_Y_S.dae
- link L_UINDEX_S: geometry collision mesh filename=package://jvrc_description/meshes/L_UINDEX_S.dae; visual mesh filename=package://jvrc_description/meshes/L_UINDEX_S.dae
- link L_ULITTLE_S: geometry collision mesh filename=package://jvrc_description/meshes/L_ULITTLE_S.dae; visual mesh filename=package://jvrc_description/meshes/L_ULITTLE_S.dae
- link L_UTHUMB_S: geometry collision mesh filename=package://jvrc_description/meshes/L_UTHUMB_S.dae; visual mesh filename=package://jvrc_description/meshes/L_UTHUMB_S.dae
- link L_WRIST_Y_S: geometry collision mesh filename=package://jvrc_description/meshes/L_WRIST_Y_S.dae; visual mesh filename=package://jvrc_description/meshes/L_WRIST_Y_S.dae
- link NECK_P_S: geometry collision mesh filename=package://jvrc_description/meshes/NECK_P_S.dae; visual mesh filename=package://jvrc_description/meshes/NECK_P_S.dae
- link NECK_Y_S: geometry collision mesh filename=package://jvrc_description/meshes/NECK_Y_S.dae; visual mesh filename=package://jvrc_description/meshes/NECK_Y_S.dae
- link PELVIS_S: geometry collision mesh filename=package://jvrc_description/meshes/PELVIS_S.dae; visual mesh filename=package://jvrc_description/meshes/PELVIS_S.dae
- link R_ANKLE_P_S: geometry collision mesh filename=package://jvrc_description/meshes/R_ANKLE_P_S.dae; visual mesh filename=package://jvrc_description/meshes/R_ANKLE_P_S.dae
- link R_ELBOW_P_S: geometry collision mesh filename=package://jvrc_description/meshes/R_ELBOW_P_S.dae; visual mesh filename=package://jvrc_description/meshes/R_ELBOW_P_S.dae
- link R_ELBOW_Y_S: geometry collision mesh filename=package://jvrc_description/meshes/R_ELBOW_Y_S.dae; visual mesh filename=package://jvrc_description/meshes/R_ELBOW_Y_S.dae
- link R_HIP_R_S: geometry collision mesh filename=package://jvrc_description/meshes/R_HIP_R_S.dae; visual mesh filename=package://jvrc_description/meshes/R_HIP_R_S.dae
- link R_HIP_Y_S: geometry collision mesh filename=package://jvrc_description/meshes/R_HIP_Y_S.dae; visual mesh filename=package://jvrc_description/meshes/R_HIP_Y_S.dae
- link R_KNEE_S: geometry collision mesh filename=package://jvrc_description/meshes/R_KNEE_S.dae; visual mesh filename=package://jvrc_description/meshes/R_KNEE_S.dae
- link R_LINDEX_S: geometry collision mesh filename=package://jvrc_description/meshes/R_LINDEX_S.dae; visual mesh filename=package://jvrc_description/meshes/R_LINDEX_S.dae
- link R_LLITTLE_S: geometry collision mesh filename=package://jvrc_description/meshes/R_LLITTLE_S.dae; visual mesh filename=package://jvrc_description/meshes/R_LLITTLE_S.dae
- link R_LTHUMB_S: geometry collision mesh filename=package://jvrc_description/meshes/R_LTHUMB_S.dae; visual mesh filename=package://jvrc_description/meshes/R_LTHUMB_S.dae
- link R_SHOULDER_P_S: geometry collision mesh filename=package://jvrc_description/meshes/R_SHOULDER_P_S.dae; visual mesh filename=package://jvrc_description/meshes/R_SHOULDER_P_S.dae
- link R_SHOULDER_Y_S: geometry collision mesh filename=package://jvrc_description/meshes/R_SHOULDER_Y_S.dae; visual mesh filename=package://jvrc_description/meshes/R_SHOULDER_Y_S.dae
- link R_UINDEX_S: geometry collision mesh filename=package://jvrc_description/meshes/R_UINDEX_S.dae; visual mesh filename=package://jvrc_description/meshes/R_UINDEX_S.dae
- link R_ULITTLE_S: geometry collision mesh filename=package://jvrc_description/meshes/R_ULITTLE_S.dae; visual mesh filename=package://jvrc_description/meshes/R_ULITTLE_S.dae
- link R_UTHUMB_S: geometry collision mesh filename=package://jvrc_description/meshes/R_UTHUMB_S.dae; visual mesh filename=package://jvrc_description/meshes/R_UTHUMB_S.dae
- link R_WRIST_Y_S: geometry collision mesh filename=package://jvrc_description/meshes/R_WRIST_Y_S.dae; visual mesh filename=package://jvrc_description/meshes/R_WRIST_Y_S.dae
- link WAIST_R_S: geometry collision mesh filename=package://jvrc_description/meshes/WAIST_R_S.dae; visual mesh filename=package://jvrc_description/meshes/WAIST_R_S.dae
- link WAIST_Y_S: geometry collision mesh filename=package://jvrc_description/meshes/WAIST_Y_S.dae; visual mesh filename=package://jvrc_description/meshes/WAIST_Y_S.dae

Commit message: Standing robot

File: jvrc_description/urdf/jvrc1.urdf (robot description, URDF)
Before this commit: robot jvrc1, 60 links, 59 joints
Links:
- removed link L_ANKLE_P_S
- removed link L_ANKLE_R_S
- removed link L_ELBOW_P_S
- removed link L_ELBOW_Y_S
- removed link L_HIP_P_S
- removed link L_HIP_R_S
- removed link L_HIP_Y_S
- removed link L_KNEE_S
- removed link L_LINDEX_S
- removed link L_LLITTLE_S
- removed link L_LTHUMB_S
- removed link L_SHOULDER_P_S
- removed link L_SHOULDER_R_S
- removed link L_SHOULDER_Y_S
- removed link L_UINDEX_S
- removed link L_ULITTLE_S
- removed link L_UTHUMB_S
- removed link L_WRIST_R_S
- removed link L_WRIST_Y_S
- removed link NECK_P_S
- removed link NECK_R_S
- removed link NECK_Y_S
- removed link PELVIS_S
- removed link R_ANKLE_P_S
- removed link R_ANKLE_R_S
- removed link R_ELBOW_P_S
- removed link R_ELBOW_Y_S
- removed link R_HIP_P_S
- removed link R_HIP_R_S
- removed link R_HIP_Y_S
- removed link R_KNEE_S
- removed link R_LINDEX_S
- removed link R_LLITTLE_S
- removed link R_LTHUMB_S
- removed link R_SHOULDER_P_S
- removed link R_SHOULDER_R_S
- removed link R_SHOULDER_Y_S
- removed link R_UINDEX_S
- removed link R_ULITTLE_S
- removed link R_UTHUMB_S
- removed link R_WRIST_R_S
- removed link R_WRIST_Y_S
- removed link WAIST_P_S
- removed link WAIST_R_S
- removed link WAIST_Y_S
- removed link base_link
- removed link dcamera
- removed link gsensor
- removed link gyrometer
- removed link l_ankle
- removed link l_wrist
- removed link lcamera
- removed link lfsensor
- removed link lhsensor
- removed link r_ankle
- removed link r_wrist
- removed link ranger
- removed link rcamera
- removed link rfsensor
- removed link rhsensor
- added link d435_link
- added link head_link, mass 1.036; collision mesh filename=meshes/head_link.STL; visual mesh filename=meshes/head_link.STL
- added link imu_in_pelvis
- added link imu_in_torso
- added link left_ankle_pitch_link, mass 0.074; collision mesh filename=meshes/left_ankle_pitch_link.STL; visual mesh filename=meshes/left_ankle_pitch_link.STL
- added link left_ankle_roll_link, mass 0.608; collision sphere radius=0.005; collision sphere radius=0.005
- added link left_elbow_link, mass 0.6; collision mesh filename=meshes/left_elbow_link.STL; visual mesh filename=meshes/left_elbow_link.STL
- added link left_hip_pitch_link, mass 1.35; collision mesh filename=meshes/left_hip_pitch_link.STL; visual mesh filename=meshes/left_hip_pitch_link.STL
- added link left_hip_roll_link, mass 1.52; collision mesh filename=meshes/left_hip_roll_link.STL; visual mesh filename=meshes/left_hip_roll_link.STL
- added link left_hip_yaw_link, mass 1.702; collision mesh filename=meshes/left_hip_yaw_link.STL; visual mesh filename=meshes/left_hip_yaw_link.STL
- added link left_knee_link, mass 1.932; collision mesh filename=meshes/left_knee_link.STL; visual mesh filename=meshes/left_knee_link.STL
- added link left_rubber_hand, mass 0.170; visual mesh filename=meshes/left_rubber_hand.STL
- added link left_shoulder_pitch_link, mass 0.718; collision cylinder length=0.05 radius=0.03; visual mesh filename=meshes/left_shoulder_pitch_link.STL
- added link left_shoulder_roll_link, mass 0.643; collision cylinder length=0.03 radius=0.03; visual mesh filename=meshes/left_shoulder_roll_link.STL
- added link left_shoulder_yaw_link, mass 0.734; collision mesh filename=meshes/left_shoulder_yaw_link.STL; visual mesh filename=meshes/left_shoulder_yaw_link.STL
- added link left_wrist_pitch_link, mass 0.48404956; collision mesh filename=meshes/left_wrist_pitch_link.STL; visual mesh filename=meshes/left_wrist_pitch_link.STL
- added link left_wrist_roll_link, mass 0.08544498; collision mesh filename=meshes/left_wrist_roll_link.STL; visual mesh filename=meshes/left_wrist_roll_link.STL
- added link left_wrist_yaw_link, mass 0.08457647; collision mesh filename=meshes/left_wrist_yaw_link.STL; visual mesh filename=meshes/left_wrist_yaw_link.STL
- added link logo_link, mass 0.001; collision mesh filename=meshes/logo_link.STL; visual mesh filename=meshes/logo_link.STL
- added link mid360_link
- added link pelvis, mass 3.813; visual mesh filename=meshes/pelvis.STL
- added link pelvis_contour_link, mass 0.001; collision mesh filename=meshes/pelvis_contour_link.STL; visual mesh filename=meshes/pelvis_contour_link.STL
- added link right_ankle_pitch_link, mass 0.074; collision mesh filename=meshes/right_ankle_pitch_link.STL; visual mesh filename=meshes/right_ankle_pitch_link.STL
- added link right_ankle_roll_link, mass 0.608; collision sphere radius=0.005; collision sphere radius=0.005
- added link right_elbow_link, mass 0.6; collision mesh filename=meshes/right_elbow_link.STL; visual mesh filename=meshes/right_elbow_link.STL
- added link right_hip_pitch_link, mass 1.35; collision mesh filename=meshes/right_hip_pitch_link.STL; visual mesh filename=meshes/right_hip_pitch_link.STL
- added link right_hip_roll_link, mass 1.52; collision mesh filename=meshes/right_hip_roll_link.STL; visual mesh filename=meshes/right_hip_roll_link.STL
- added link right_hip_yaw_link, mass 1.702; collision mesh filename=meshes/right_hip_yaw_link.STL; visual mesh filename=meshes/right_hip_yaw_link.STL
- added link right_knee_link, mass 1.932; collision mesh filename=meshes/right_knee_link.STL; visual mesh filename=meshes/right_knee_link.STL
- added link right_rubber_hand, mass 0.170; visual mesh filename=meshes/right_rubber_hand.STL
- added link right_shoulder_pitch_link, mass 0.718; collision cylinder length=0.05 radius=0.03; visual mesh filename=meshes/right_shoulder_pitch_link.STL
- added link right_shoulder_roll_link, mass 0.643; collision cylinder length=0.03 radius=0.03; visual mesh filename=meshes/right_shoulder_roll_link.STL
- added link right_shoulder_yaw_link, mass 0.734; collision mesh filename=meshes/right_shoulder_yaw_link.STL; visual mesh filename=meshes/right_shoulder_yaw_link.STL
- added link right_wrist_pitch_link, mass 0.48404956; collision mesh filename=meshes/right_wrist_pitch_link.STL; visual mesh filename=meshes/right_wrist_pitch_link.STL
- added link right_wrist_roll_link, mass 0.08544498; collision mesh filename=meshes/right_wrist_roll_link.STL; visual mesh filename=meshes/right_wrist_roll_link.STL
- added link right_wrist_yaw_link, mass 0.08457647; collision mesh filename=meshes/right_wrist_yaw_link.STL; visual mesh filename=meshes/right_wrist_yaw_link.STL
- added link torso_link, mass 6.78; collision mesh filename=meshes/torso_link_rev_1_0.STL; visual mesh filename=meshes/torso_link_rev_1_0.STL
- added link waist_roll_link, mass 0.086; visual mesh filename=meshes/waist_roll_link_rev_1_0.STL
- added link waist_yaw_link, mass 0.214; visual mesh filename=meshes/waist_yaw_link_rev_1_0.STL
Joints:
- removed joint L_ANKLE_P
- removed joint L_ANKLE_R
- removed joint L_ELBOW_P
- removed joint L_ELBOW_Y
- removed joint L_HIP_P
- removed joint L_HIP_R
- removed joint L_HIP_Y
- removed joint L_KNEE
- removed joint L_LINDEX
- removed joint L_LLITTLE
- removed joint L_LTHUMB
- removed joint L_SHOULDER_P
- removed joint L_SHOULDER_R
- removed joint L_SHOULDER_Y
- removed joint L_UINDEX
- removed joint L_ULITTLE
- removed joint L_UTHUMB
- removed joint L_WRIST_R
- removed joint L_WRIST_Y
- removed joint NECK_P
- removed joint NECK_R
- removed joint NECK_Y
- removed joint R_ANKLE_P
- removed joint R_ANKLE_R
- removed joint R_ELBOW_P
- removed joint R_ELBOW_Y
- removed joint R_HIP_P
- removed joint R_HIP_R
- removed joint R_HIP_Y
- removed joint R_KNEE
- removed joint R_LINDEX
- removed joint R_LLITTLE
- removed joint R_LTHUMB
- removed joint R_SHOULDER_P
- removed joint R_SHOULDER_R
- removed joint R_SHOULDER_Y
- removed joint R_UINDEX
- removed joint R_ULITTLE
- removed joint R_UTHUMB
- removed joint R_WRIST_R
- removed joint R_WRIST_Y
- removed joint WAIST_P
- removed joint WAIST_R
- removed joint WAIST_Y
- removed joint dcamera_JOINT
- removed joint gsensor_JOINT
- removed joint gyrometer_JOINT
- removed joint l_ankle_joint
- removed joint l_wrist_joint
- removed joint lcamera_JOINT
- removed joint lfsensor_JOINT
- removed joint lhsensor_JOINT
- removed joint r_ankle_joint
- removed joint r_wrist_joint
- removed joint ranger_JOINT
- removed joint rcamera_JOINT
- removed joint rfsensor_JOINT
- removed joint rhsensor_JOINT
- removed joint waist
- added joint d435_joint: type fixed, parent torso_link, child d435_link, origin xyz=0.0576235 0.01753 0.42987 rpy=0 0.8307767239493009 0
- added joint head_joint: type fixed, parent torso_link, child head_link, origin xyz=0.0039635 0 -0.044 rpy=0 0 0
- added joint imu_in_pelvis_joint: type fixed, parent pelvis, child imu_in_pelvis, origin xyz=0.04525 0 -0.08339 rpy=0 0 0
- added joint imu_in_torso_joint: type fixed, parent torso_link, child imu_in_torso, origin xyz=-0.03959 -0.00224 0.14792 rpy=0 0 0
- added joint left_ankle_pitch_joint: type revolute, parent left_knee_link, child left_ankle_pitch_link, origin xyz=0 -9.4445E-05 -0.30001 rpy=0 0 0, axis 0 1 0, limit lower=-0.87267 upper=0.5236 effort=35 velocity=30
- added joint left_ankle_roll_joint: type revolute, parent left_ankle_pitch_link, child left_ankle_roll_link, origin xyz=0 0 -0.017558 rpy=0 0 0, axis 1 0 0, limit lower=-0.2618 upper=0.2618 effort=35 velocity=30
- added joint left_elbow_joint: type revolute, parent left_shoulder_yaw_link, child left_elbow_link, origin xyz=0.015783 0 -0.080518 rpy=0 0 0, axis 0 1 0, limit lower=-1.0472 upper=2.0944 effort=25 velocity=37
- added joint left_hand_palm_joint: type fixed, parent left_wrist_yaw_link, child left_rubber_hand, origin xyz=0.0415 0.003 0 rpy=0 0 0
- added joint left_hip_pitch_joint: type revolute, parent pelvis, child left_hip_pitch_link, origin xyz=0 0.064452 -0.1027 rpy=0 0 0, axis 0 1 0, limit lower=-2.5307 upper=2.8798 effort=88 velocity=32
- added joint left_hip_roll_joint: type revolute, parent left_hip_pitch_link, child left_hip_roll_link, origin xyz=0 0.052 -0.030465 rpy=0 -0.1749 0, axis 1 0 0, limit lower=-0.5236 upper=2.9671 effort=139 velocity=20
- added joint left_hip_yaw_joint: type revolute, parent left_hip_roll_link, child left_hip_yaw_link, origin xyz=0.025001 0 -0.12412 rpy=0 0 0, axis 0 0 1, limit lower=-2.7576 upper=2.7576 effort=88 velocity=32
- added joint left_knee_joint: type revolute, parent left_hip_yaw_link, child left_knee_link, origin xyz=-0.078273 0.0021489 -0.17734 rpy=0 0.1749 0, axis 0 1 0, limit lower=-0.087267 upper=2.8798 effort=139 velocity=20
- added joint left_shoulder_pitch_joint: type revolute, parent torso_link, child left_shoulder_pitch_link, origin xyz=0.0039563 0.10022 0.24778 rpy=0.27931 5.4949E-05 -0.00019159, axis 0 1 0, limit lower=-3.0892 upper=2.6704 effort=25 velocity=37
- added joint left_shoulder_roll_joint: type revolute, parent left_shoulder_pitch_link, child left_shoulder_roll_link, origin xyz=0 0.038 -0.013831 rpy=-0.27925 0 0, axis 1 0 0, limit lower=-1.5882 upper=2.2515 effort=25 velocity=37
- added joint left_shoulder_yaw_joint: type revolute, parent left_shoulder_roll_link, child left_shoulder_yaw_link, origin xyz=0 0.00624 -0.1032 rpy=0 0 0, axis 0 0 1, limit lower=-2.618 upper=2.618 effort=25 velocity=37
- added joint left_wrist_pitch_joint: type revolute, parent left_wrist_roll_link, child left_wrist_pitch_link, origin xyz=0.038 0 0 rpy=0 0 0, axis 0 1 0, limit lower=-1.614429558 upper=1.614429558 effort=5 velocity=22
- added joint left_wrist_roll_joint: type revolute, parent left_elbow_link, child left_wrist_roll_link, origin xyz=0.100 0.00188791 -0.010 rpy=0 0 0, axis 1 0 0, limit lower=-1.972222054 upper=1.972222054 effort=25 velocity=37
- added joint left_wrist_yaw_joint: type revolute, parent left_wrist_pitch_link, child left_wrist_yaw_link, origin xyz=0.046 0 0 rpy=0 0 0, axis 0 0 1, limit lower=-1.614429558 upper=1.614429558 effort=5 velocity=22
- added joint logo_joint: type fixed, parent torso_link, child logo_link, origin xyz=0.0039635 0 -0.044 rpy=0 0 0
- added joint mid360_joint: type fixed, parent torso_link, child mid360_link, origin xyz=0.0002835 0.00003 0.41618 rpy=0 0.04014257279586953 0
- added joint pelvis_contour_joint: type fixed, parent pelvis, child pelvis_contour_link
- added joint right_ankle_pitch_joint: type revolute, parent right_knee_link, child right_ankle_pitch_link, origin xyz=0 9.4445E-05 -0.30001 rpy=0 0 0, axis 0 1 0, limit lower=-0.87267 upper=0.5236 effort=35 velocity=30
- added joint right_ankle_roll_joint: type revolute, parent right_ankle_pitch_link, child right_ankle_roll_link, origin xyz=0 0 -0.017558 rpy=0 0 0, axis 1 0 0, limit lower=-0.2618 upper=0.2618 effort=35 velocity=30
- added joint right_elbow_joint: type revolute, parent right_shoulder_yaw_link, child right_elbow_link, origin xyz=0.015783 0 -0.080518 rpy=0 0 0, axis 0 1 0, limit lower=-1.0472 upper=2.0944 effort=25 velocity=37
- added joint right_hand_palm_joint: type fixed, parent right_wrist_yaw_link, child right_rubber_hand, origin xyz=0.0415 -0.003 0 rpy=0 0 0
- added joint right_hip_pitch_joint: type revolute, parent pelvis, child right_hip_pitch_link, origin xyz=0 -0.064452 -0.1027 rpy=0 0 0, axis 0 1 0, limit lower=-2.5307 upper=2.8798 effort=88 velocity=32
- added joint right_hip_roll_joint: type revolute, parent right_hip_pitch_link, child right_hip_roll_link, origin xyz=0 -0.052 -0.030465 rpy=0 -0.1749 0, axis 1 0 0, limit lower=-2.9671 upper=0.5236 effort=139 velocity=20
- added joint right_hip_yaw_joint: type revolute, parent right_hip_roll_link, child right_hip_yaw_link, origin xyz=0.025001 0 -0.12412 rpy=0 0 0, axis 0 0 1, limit lower=-2.7576 upper=2.7576 effort=88 velocity=32
- added joint right_knee_joint: type revolute, parent right_hip_yaw_link, child right_knee_link, origin xyz=-0.078273 -0.0021489 -0.17734 rpy=0 0.1749 0, axis 0 1 0, limit lower=-0.087267 upper=2.8798 effort=139 velocity=20
- added joint right_shoulder_pitch_joint: type revolute, parent torso_link, child right_shoulder_pitch_link, origin xyz=0.0039563 -0.10021 0.24778 rpy=-0.27931 5.4949E-05 0.00019159, axis 0 1 0, limit lower=-3.0892 upper=2.6704 effort=25 velocity=37
- added joint right_shoulder_roll_joint: type revolute, parent right_shoulder_pitch_link, child right_shoulder_roll_link, origin xyz=0 -0.038 -0.013831 rpy=0.27925 0 0, axis 1 0 0, limit lower=-2.2515 upper=1.5882 effort=25 velocity=37
- added joint right_shoulder_yaw_joint: type revolute, parent right_shoulder_roll_link, child right_shoulder_yaw_link, origin xyz=0 -0.00624 -0.1032 rpy=0 0 0, axis 0 0 1, limit lower=-2.618 upper=2.618 effort=25 velocity=37
- added joint right_wrist_pitch_joint: type revolute, parent right_wrist_roll_link, child right_wrist_pitch_link, origin xyz=0.038 0 0 rpy=0 0 0, axis 0 1 0, limit lower=-1.614429558 upper=1.614429558 effort=5 velocity=22
- added joint right_wrist_roll_joint: type revolute, parent right_elbow_link, child right_wrist_roll_link, origin xyz=0.100 -0.00188791 -0.010 rpy=0 0 0, axis 1 0 0, limit lower=-1.972222054 upper=1.972222054 effort=25 velocity=37
- added joint right_wrist_yaw_joint: type revolute, parent right_wrist_pitch_link, child right_wrist_yaw_link, origin xyz=0.046 0 0 rpy=0 0 0, axis 0 0 1, limit lower=-1.614429558 upper=1.614429558 effort=5 velocity=22
- added joint waist_pitch_joint: type revolute, parent waist_roll_link, child torso_link, origin xyz=0 0 0 rpy=0 0 0, axis 0 1 0, limit lower=-0.52 upper=0.52 effort=35 velocity=30
- added joint waist_roll_joint: type revolute, parent waist_yaw_link, child waist_roll_link, origin xyz=-0.0039635 0 0.044 rpy=0 0 0, axis 1 0 0, limit lower=-0.52 upper=0.52 effort=35 velocity=30
- added joint waist_yaw_joint: type revolute, parent pelvis, child waist_yaw_link, origin xyz=0 0 0 rpy=0 0 0, axis 0 0 1, limit lower=-2.618 upper=2.618 effort=88 velocity=32
