Commit message: Added plots

File: jvrc_description/urdf/jvrc1.urdf (robot description, URDF)
Before this commit: robot jvrc1, 39 links, 38 joints
Links:
- removed link d435_link
- removed link head_link
- removed link imu_in_pelvis
- removed link imu_in_torso
- removed link left_ankle_pitch_link
- removed link left_ankle_roll_link
- removed link left_elbow_link
- removed link left_hip_pitch_link
- removed link left_hip_roll_link
- removed link left_hip_yaw_link
- removed link left_knee_link
- removed link left_rubber_hand
- removed link left_shoulder_pitch_link
- removed link left_shoulder_roll_link
- removed link left_shoulder_yaw_link
- removed link left_wrist_pitch_link
- removed link left_wrist_roll_link
- removed link left_wrist_yaw_link
- removed link logo_link
- removed link mid360_link
- removed link pelvis
- removed link pelvis_contour_link
- removed link right_ankle_pitch_link
- removed link right_ankle_roll_link
- removed link right_elbow_link
- removed link right_hip_pitch_link
- removed link right_hip_roll_link
- removed link right_hip_yaw_link
- removed link right_knee_link
- removed link right_rubber_hand
- removed link right_shoulder_pitch_link
- removed link right_shoulder_roll_link
- removed link right_shoulder_yaw_link
- removed link right_wrist_pitch_link
- removed link right_wrist_roll_link
- removed link right_wrist_yaw_link
- removed link torso_link
- removed link waist_roll_link
- removed link waist_yaw_link
- added link L_ANKLE_P_S, mass 1.5; collision mesh filename=package://jvrc_description/meshes/L_ANKLE_P_S.dae; visual mesh filename=package://jvrc_description/meshes/L_ANKLE_P_S.dae
- added link L_ANKLE_R_S, mass 1.0
- added link L_ELBOW_P_S, mass 1.0; collision mesh filename=package://jvrc_description/meshes/L_ELBOW_P_S.dae; visual mesh filename=package://jvrc_description/meshes/L_ELBOW_P_S.dae
- added link L_ELBOW_Y_S, mass 1.0; collision mesh filename=package://jvrc_description/meshes/L_ELBOW_Y_S.dae; visual mesh filename=package://jvrc_description/meshes/L_ELBOW_Y_S.dae
- added link L_HIP_P_S, mass 1.0
- added link L_HIP_R_S, mass 1.0; collision mesh filename=package://jvrc_description/meshes/L_HIP_R_S.dae; visual mesh filename=package://jvrc_description/meshes/L_HIP_R_S.dae
- added link L_HIP_Y_S, mass 3.0; collision mesh filename=package://jvrc_description/meshes/L_HIP_Y_S.dae; visual mesh filename=package://jvrc_description/meshes/L_HIP_Y_S.dae
- added link L_KNEE_S, mass 3.0; collision mesh filename=package://jvrc_description/meshes/L_KNEE_S.dae; visual mesh filename=package://jvrc_description/meshes/L_KNEE_S.dae
- added link L_LINDEX_S, mass 0.2; collision mesh filename=package://jvrc_description/meshes/L_LINDEX_S.dae; visual mesh filename=package://jvrc_description/meshes/L_LINDEX_S.dae
- added link L_LLITTLE_S, mass 0.2; collision mesh filename=package://jvrc_description/meshes/L_LLITTLE_S.dae; visual mesh filename=package://jvrc_description/meshes/L_LLITTLE_S.dae
- added link L_LTHUMB_S, mass 0.2; collision mesh filename=package://jvrc_description/meshes/L_LTHUMB_S.dae; visual mesh filename=package://jvrc_description/meshes/L_LTHUMB_S.dae
- added link L_SHOULDER_P_S, mass 1.0; collision mesh filename=package://jvrc_description/meshes/L_SHOULDER_P_S.dae; visual mesh filename=package://jvrc_description/meshes/L_SHOULDER_P_S.dae
- added link L_SHOULDER_R_S, mass 1.0
- added link L_SHOULDER_Y_S, mass 2.0; collision mesh filename=package://jvrc_description/meshes/L_SHOULDER_Y_S.dae; visual mesh filename=package://jvrc_description/meshes/L_SHOULDER_Y_S.dae
- added link L_UINDEX_S, mass 0.2; collision mesh filename=package://jvrc_description/meshes/L_UINDEX_S.dae; visual mesh filename=package://jvrc_description/meshes/L_UINDEX_S.dae
- added link L_ULITTLE_S, mass 0.2; collision mesh filename=package://jvrc_description/meshes/L_ULITTLE_S.dae; visual mesh filename=package://jvrc_description/meshes/L_ULITTLE_S.dae
- added link L_UTHUMB_S, mass 0.2; collision mesh filename=package://jvrc_description/meshes/L_UTHUMB_S.dae; visual mesh filename=package://jvrc_description/meshes/L_UTHUMB_S.dae
- added link L_WRIST_R_S, mass 0.5
- added link L_WRIST_Y_S, mass 0.5; collision mesh filename=package://jvrc_description/meshes/L_WRIST_Y_S.dae; visual mesh filename=package://jvrc_description/meshes/L_WRIST_Y_S.dae
- added link NECK_P_S, mass 2.0; collision mesh filename=package://jvrc_description/meshes/NECK_P_S.dae; visual mesh filename=package://jvrc_description/meshes/NECK_P_S.dae
- added link NECK_R_S, mass 0.5
- added link NECK_Y_S, mass 0.5; collision mesh filename=package://jvrc_description/meshes/NECK_Y_S.dae; visual mesh filename=package://jvrc_description/meshes/NECK_Y_S.dae
- added link PELVIS_S, mass 10.0; collision mesh filename=package://jvrc_description/meshes/PELVIS_S.dae; visual mesh filename=package://jvrc_description/meshes/PELVIS_S.dae
- added link R_ANKLE_P_S, mass 1.5; collision mesh filename=package://jvrc_description/meshes/R_ANKLE_P_S.dae; visual mesh filename=package://jvrc_description/meshes/R_ANKLE_P_S.dae
- added link R_ANKLE_R_S, mass 1.0
- added link R_ELBOW_P_S, mass 1.0; collision mesh filename=package://jvrc_description/meshes/R_ELBOW_P_S.dae; visual mesh filename=package://jvrc_description/meshes/R_ELBOW_P_S.dae
- added link R_ELBOW_Y_S, mass 1.0; collision mesh filename=package://jvrc_description/meshes/R_ELBOW_Y_S.dae; visual mesh filename=package://jvrc_description/meshes/R_ELBOW_Y_S.dae
- added link R_HIP_P_S, mass 1.0
- added link R_HIP_R_S, mass 1.0; collision mesh filename=package://jvrc_description/meshes/R_HIP_R_S.dae; visual mesh filename=package://jvrc_description/meshes/R_HIP_R_S.dae
- added link R_HIP_Y_S, mass 3.0; collision mesh filename=package://jvrc_description/meshes/R_HIP_Y_S.dae; visual mesh filename=package://jvrc_description/meshes/R_HIP_Y_S.dae
- added link R_KNEE_S, mass 3.0; collision mesh filename=package://jvrc_description/meshes/R_KNEE_S.dae; visual mesh filename=package://jvrc_description/meshes/R_KNEE_S.dae
- added link R_LINDEX_S, mass 0.2; collision mesh filename=package://jvrc_description/meshes/R_LINDEX_S.dae; visual mesh filename=package://jvrc_description/meshes/R_LINDEX_S.dae
- added link R_LLITTLE_S, mass 0.2; collision mesh filename=package://jvrc_description/meshes/R_LLITTLE_S.dae; visual mesh filename=package://jvrc_description/meshes/R_LLITTLE_S.dae
- added link R_LTHUMB_S, mass 0.2; collision mesh filename=package://jvrc_description/meshes/R_LTHUMB_S.dae; visual mesh filename=package://jvrc_description/meshes/R_LTHUMB_S.dae
- added link R_SHOULDER_P_S, mass 1.0; collision mesh filename=package://jvrc_description/meshes/R_SHOULDER_P_S.dae; visual mesh filename=package://jvrc_description/meshes/R_SHOULDER_P_S.dae
- added link R_SHOULDER_R_S, mass 1.0
- added link R_SHOULDER_Y_S, mass 2.0; collision mesh filename=package://jvrc_description/meshes/R_SHOULDER_Y_S.dae; visual mesh filename=package://jvrc_description/meshes/R_SHOULDER_Y_S.dae
- added link R_UINDEX_S, mass 0.2; collision mesh filename=package://jvrc_description/meshes/R_UINDEX_S.dae; visual mesh filename=package://jvrc_description/meshes/R_UINDEX_S.dae
- added link R_ULITTLE_S, mass 0.2; collision mesh filename=package://jvrc_description/meshes/R_ULITTLE_S.dae; visual mesh filename=package://jvrc_description/meshes/R_ULITTLE_S.dae
- added link R_UTHUMB_S, mass 0.2; collision mesh filename=package://jvrc_description/meshes/R_UTHUMB_S.dae; visual mesh filename=package://jvrc_description/meshes/R_UTHUMB_S.dae
- added link R_WRIST_R_S, mass 0.5
- added link R_WRIST_Y_S, mass 0.5; collision mesh filename=package://jvrc_description/meshes/R_WRIST_Y_S.dae; visual mesh filename=package://jvrc_description/meshes/R_WRIST_Y_S.dae
- added link WAIST_P_S, mass 1.0
- added link WAIST_R_S, mass 10.0; collision mesh filename=package://jvrc_description/meshes/WAIST_R_S.dae; visual mesh filename=package://jvrc_description/meshes/WAIST_R_S.dae
- added link WAIST_Y_S, mass 1.0; collision mesh filename=package://jvrc_description/meshes/WAIST_Y_S.dae; visual mesh filename=package://jvrc_description/meshes/WAIST_Y_S.dae
- added link base_link
- added link dcamera
- added link gsensor
- added link gyrometer
- added link l_ankle
- added link l_wrist
- added link lcamera
- added link lfsensor
- added link lhsensor
- added link r_ankle
- added link r_wrist
- added link ranger
- added link rcamera
- added link rfsensor
- added link rhsensor
Joints:
- removed joint d435_joint
- removed joint head_joint
- removed joint imu_in_pelvis_joint
- removed joint imu_in_torso_joint
- removed joint left_ankle_pitch_joint
- removed joint left_ankle_roll_joint
- removed joint left_elbow_joint
- removed joint left_hand_palm_joint
- removed joint left_hip_pitch_joint
- removed joint left_hip_roll_joint
- removed joint left_hip_yaw_joint
- removed joint left_knee_joint
- removed joint left_shoulder_pitch_joint
- removed joint left_shoulder_roll_joint
- removed joint left_shoulder_yaw_joint
- removed joint left_wrist_pitch_joint
- removed joint left_wrist_roll_joint
- removed joint left_wrist_yaw_joint
- removed joint logo_joint
- removed joint mid360_joint
- removed joint pelvis_contour_joint
- removed joint right_ankle_pitch_joint
- removed joint right_ankle_roll_joint
- removed joint right_elbow_joint
- removed joint right_hand_palm_joint
- removed joint right_hip_pitch_joint
- removed joint right_hip_roll_joint
- removed joint right_hip_yaw_joint
- removed joint right_knee_joint
- removed joint right_shoulder_pitch_joint
- removed joint right_shoulder_roll_joint
- removed joint right_shoulder_yaw_joint
- removed joint right_wrist_pitch_joint
- removed joint right_wrist_roll_joint
- removed joint right_wrist_yaw_joint
- removed joint waist_pitch_joint
- removed joint waist_roll_joint
- removed joint waist_yaw_joint
- added joint L_ANKLE_P: type revolute, parent L_ANKLE_R_S, child L_ANKLE_P_S, origin xyz=-4.85722573274e-17 3.60822483003e-16 -2.22044604925e-16 rpy=0.0 -0.0 0.0, axis 0.0 1.0 0.0, limit lower=-1.4835298642 upper=0.959931088597 effort=100.0 velocity=14.18435
- added joint L_ANKLE_R: type revolute, parent L_KNEE_S, child L_ANKLE_R_S, origin xyz=0.04 1.52655665886e-16 -0.357 rpy=0.0 -0.0 0.0, axis 1.0 0.0 0.0, limit lower=-0.785398163397 upper=0.610865238198 effort=100.0 velocity=15.18435
- added joint L_ELBOW_P: type revolute, parent L_SHOULDER_Y_S, child L_ELBOW_P_S, origin xyz=0.004 -2.77555756156e-17 -0.305 rpy=0.0 -0.0 0.0, axis 0.0 1.0 0.0, limit lower=-2.53072741539 upper=0.0 effort=100.0 velocity=9.42477
- added joint L_ELBOW_Y: type revolute, parent L_ELBOW_P_S, child L_ELBOW_Y_S, origin xyz=-0.004 3.88578058619e-16 -0.239 rpy=0.0 -0.0 0.0, axis 0.0 0.0 1.0, limit lower=-1.91986217719 upper=1.91986217719 effort=100.0 velocity=3.66519
- added joint L_HIP_P: type revolute, parent PELVIS_S, child L_HIP_P_S, origin xyz=0.0 0.096 0.0 rpy=0.0 -0.0 0.0, axis 0.0 1.0 0.0, limit lower=-2.09439510239 upper=0.785398163397 effort=100.0 velocity=12.56636
- added joint L_HIP_R: type revolute, parent L_HIP_P_S, child L_HIP_R_S, origin xyz=0.0 -2.77555756156e-17 0.0 rpy=0.0 -0.0 0.0, axis 1.0 0.0 0.0, limit lower=-0.349065850399 upper=0.785398163397 effort=100.0 velocity=8.90117
- added joint L_HIP_Y: type revolute, parent L_HIP_R_S, child L_HIP_Y_S, origin xyz=0.0 -2.77555756156e-17 0.0 rpy=0.0 -0.0 0.0, axis 0.0 0.0 1.0, limit lower=-0.785398163397 upper=0.523598775598 effort=100.0 velocity=8.90117
- added joint L_KNEE: type revolute, parent L_HIP_Y_S, child L_KNEE_S, origin xyz=-0.02 -2.77555756156e-17 -0.389 rpy=0.0 -0.0 0.0, axis 0.0 1.0 0.0, limit lower=0.0 upper=2.61799387799 effort=100.0 velocity=14.66075
- added joint L_LINDEX: type revolute, parent L_UINDEX_S, child L_LINDEX_S, origin xyz=3.46944695195e-17 1.38777878078e-16 -0.045 rpy=0.0 -0.0 0.0, axis 1.0 0.0 0.0, limit lower=-1.57079632679 upper=0.0 effort=100.0 velocity=5.75958, mimic joint=L_UTHUMB multiplier=-2 offset=0
- added joint L_LLITTLE: type revolute, parent L_ULITTLE_S, child L_LLITTLE_S, origin xyz=-3.46944695195e-17 2.77555756156e-17 -0.045 rpy=0.0 -0.0 0.0, axis 1.0 0.0 0.0, limit lower=-1.57079632679 upper=0.0 effort=100.0 velocity=5.75958, mimic joint=L_UTHUMB multiplier=-2 offset=0
- added joint L_LTHUMB: type revolute, parent L_UTHUMB_S, child L_LTHUMB_S, origin xyz=0.0 2.16493489802e-15 -0.045 rpy=0.0 -0.0 0.0, axis 1.0 0.0 0.0, limit lower=-0.0 upper=1.57079632679 effort=100.0 velocity=13.6135, mimic joint=L_UTHUMB multiplier=2 offset=0
- added joint L_SHOULDER_P: type revolute, parent WAIST_R_S, child L_SHOULDER_P_S, origin xyz=0.0 0.24 0.33 rpy=0.0 -0.0 0.0, axis 0.0 1.0 0.0, limit lower=-3.14159265359 upper=1.0471975512 effort=100.0 velocity=8.90117
- added joint L_SHOULDER_R: type revolute, parent L_SHOULDER_P_S, child L_SHOULDER_R_S, origin xyz=0.0 2.77555756156e-17 -5.55111512313e-16 rpy=0.0 -0.0 0.0, axis 1.0 0.0 0.0, limit lower=-0.174532925199 upper=1.74532925199 effort=100.0 velocity=8.90117
- added joint L_SHOULDER_Y: type revolute, parent L_SHOULDER_R_S, child L_SHOULDER_Y_S, origin xyz=0.0 2.77555756156e-17 -5.55111512313e-16 rpy=0.0 -0.0 0.0, axis 0.0 0.0 1.0, limit lower=-1.57079632679 upper=1.57079632679 effort=100.0 velocity=4.18879
- added joint L_UINDEX: type revolute, parent L_WRIST_Y_S, child L_UINDEX_S, origin xyz=0.025 0.006 -0.102 rpy=0.0 -0.0 0.0, axis 1.0 0.0 0.0, limit lower=-1.57079632679 upper=0.0 effort=100.0 velocity=9.42477, mimic joint=L_UTHUMB multiplier=-2 offset=0
- added joint L_ULITTLE: type revolute, parent L_WRIST_Y_S, child L_ULITTLE_S, origin xyz=-0.025 0.006 -0.102 rpy=0.0 -0.0 0.0, axis 1.0 0.0 0.0, limit lower=-1.57079632679 upper=0.0 effort=100.0 velocity=9.42477, mimic joint=L_UTHUMB multiplier=-2 offset=0
- added joint L_UTHUMB: type revolute, parent L_WRIST_Y_S, child L_UTHUMB_S, origin xyz=0.0 -0.023 -0.084 rpy=0.0 -0.0 0.0, axis 1.0 0.0 0.0, limit lower=-0.0 upper=0.785398163397 effort=100.0 velocity=6.80678
- added joint L_WRIST_R: type revolute, parent L_ELBOW_Y_S, child L_WRIST_R_S, origin xyz=0.0 -2.77555756156e-16 -1.80411241502e-16 rpy=0.0 -0.0 0.0, axis 1.0 0.0 0.0, limit lower=-1.91986217719 upper=1.91986217719 effort=100.0 velocity=5.75958
- added joint L_WRIST_Y: type revolute, parent L_WRIST_R_S, child L_WRIST_Y_S, origin xyz=0.0 -2.77555756156e-16 -1.80411241502e-16 rpy=0.0 -0.0 0.0, axis 0.0 0.0 1.0, limit lower=-2.61799387799 upper=2.61799387799 effort=100.0 velocity=3.66519
- added joint NECK_P: type revolute, parent NECK_R_S, child NECK_P_S, origin xyz=8.23993651089e-18 0.0 2.22044604925e-16 rpy=0.0 -0.0 0.0, axis 0.0 1.0 0.0, limit lower=-0.872664625997 upper=1.0471975512 effort=100.0 velocity=5.75958
- added joint NECK_R: type revolute, parent NECK_Y_S, child NECK_R_S, origin xyz=8.23993651089e-18 0.0 2.22044604925e-16 rpy=0.0 -0.0 0.0, axis 1.0 0.0 0.0, limit lower=-0.872664625997 upper=0.872664625997 effort=100.0 velocity=5.75958
- added joint NECK_Y: type revolute, parent WAIST_R_S, child NECK_Y_S, origin xyz=-0.003 0.0 0.453 rpy=0.0 -0.0 0.0, axis 0.0 0.0 1.0, limit lower=-1.2217304764 upper=1.2217304764 effort=100.0 velocity=5.23598
- added joint R_ANKLE_P: type revolute, parent R_ANKLE_R_S, child R_ANKLE_P_S, origin xyz=-1.73472347598e-17 -4.4408920985e-16 -1.11022302463e-16 rpy=0.0 -0.0 0.0, axis 0.0 1.0 0.0, limit lower=-1.4835298642 upper=0.959931088597 effort=100.0 velocity=14.18435
- added joint R_ANKLE_R: type revolute, parent R_KNEE_S, child R_ANKLE_R_S, origin xyz=0.04 1.11022302463e-16 -0.357 rpy=0.0 -0.0 0.0, axis 1.0 0.0 0.0, limit lower=-0.610865238198 upper=0.785398163397 effort=100.0 velocity=15.18435
- added joint R_ELBOW_P: type revolute, parent R_SHOULDER_Y_S, child R_ELBOW_P_S, origin xyz=0.004 2.77555756156e-17 -0.305 rpy=0.0 -0.0 0.0, axis 0.0 1.0 0.0, limit lower=-2.53072741539 upper=0.0 effort=100.0 velocity=9.42477
- added joint R_ELBOW_Y: type revolute, parent R_ELBOW_P_S, child R_ELBOW_Y_S, origin xyz=-0.004 -4.99600361081e-16 -0.239 rpy=0.0 -0.0 0.0, axis 0.0 0.0 1.0, limit lower=-1.91986217719 upper=1.91986217719 effort=100.0 velocity=3.66519
- added joint R_HIP_P: type revolute, parent PELVIS_S, child R_HIP_P_S, origin xyz=0.0 -0.096 0.0 rpy=0.0 -0.0 0.0, axis 0.0 1.0 0.0, limit lower=-2.09439510239 upper=0.785398163397 effort=100.0 velocity=12.56636
- added joint R_HIP_R: type revolute, parent R_HIP_P_S, child R_HIP_R_S, origin xyz=0.0 2.77555756156e-17 0.0 rpy=0.0 -0.0 0.0, axis 1.0 0.0 0.0, limit lower=-0.785398163397 upper=0.349065850399 effort=100.0 velocity=8.90117
- added joint R_HIP_Y: type revolute, parent R_HIP_R_S, child R_HIP_Y_S, origin xyz=0.0 2.77555756156e-17 0.0 rpy=0.0 -0.0 0.0, axis 0.0 0.0 1.0, limit lower=-0.523598775598 upper=0.785398163397 effort=100.0 velocity=8.90117
- added joint R_KNEE: type revolute, parent R_HIP_Y_S, child R_KNEE_S, origin xyz=-0.02 2.77555756156e-17 -0.389 rpy=0.0 -0.0 0.0, axis 0.0 1.0 0.0, limit lower=0.0 upper=2.61799387799 effort=100.0 velocity=14.66075
- added joint R_LINDEX: type revolute, parent R_UINDEX_S, child R_LINDEX_S, origin xyz=3.46944695195e-17 -2.77555756156e-17 -0.045 rpy=0.0 -0.0 0.0, axis 1.0 0.0 0.0, limit lower=0.0 upper=1.57079632679 effort=100.0 velocity=5.75958, mimic joint=R_UTHUMB multiplier=-2 offset=0
- added joint R_LLITTLE: type revolute, parent R_ULITTLE_S, child R_LLITTLE_S, origin xyz=-3.46944695195e-17 -1.38777878078e-16 -0.045 rpy=0.0 -0.0 0.0, axis 1.0 0.0 0.0, limit lower=0.0 upper=1.57079632679 effort=100.0 velocity=5.75958, mimic joint=R_UTHUMB multiplier=-2 offset=0
- added joint R_LTHUMB: type revolute, parent R_UTHUMB_S, child R_LTHUMB_S, origin xyz=0.0 -2.47024622979e-15 -0.045 rpy=0.0 -0.0 0.0, axis 1.0 0.0 0.0, limit lower=-1.57079632679 upper=0.0 effort=100.0 velocity=13.6135, mimic joint=R_UTHUMB multiplier=2 offset=0
- added joint R_SHOULDER_P: type revolute, parent WAIST_R_S, child R_SHOULDER_P_S, origin xyz=0.0 -0.24 0.33 rpy=0.0 -0.0 0.0, axis 0.0 1.0 0.0, limit lower=-3.14159265359 upper=1.0471975512 effort=100.0 velocity=8.90117
- added joint R_SHOULDER_R: type revolute, parent R_SHOULDER_P_S, child R_SHOULDER_R_S, origin xyz=0.0 -2.77555756156e-17 -7.77156117238e-16 rpy=0.0 -0.0 0.0, axis 1.0 0.0 0.0, limit lower=-1.74532925199 upper=0.174532925199 effort=100.0 velocity=8.90117
- added joint R_SHOULDER_Y: type revolute, parent R_SHOULDER_R_S, child R_SHOULDER_Y_S, origin xyz=0.0 -2.77555756156e-17 -7.77156117238e-16 rpy=0.0 -0.0 0.0, axis 0.0 0.0 1.0, limit lower=-1.57079632679 upper=1.57079632679 effort=100.0 velocity=4.18879
- added joint R_UINDEX: type revolute, parent R_WRIST_Y_S, child R_UINDEX_S, origin xyz=0.025 -0.006 -0.102 rpy=0.0 -0.0 0.0, axis 1.0 0.0 0.0, limit lower=0.0 upper=1.57079632679 effort=100.0 velocity=9.42477, mimic joint=R_UTHUMB multiplier=-2 offset=0
- added joint R_ULITTLE: type revolute, parent R_WRIST_Y_S, child R_ULITTLE_S, origin xyz=-0.025 -0.006 -0.102 rpy=0.0 -0.0 0.0, axis 1.0 0.0 0.0, limit lower=0.0 upper=1.57079632679 effort=100.0 velocity=9.42477, mimic joint=R_UTHUMB multiplier=-2 offset=0
- added joint R_UTHUMB: type revolute, parent R_WRIST_Y_S, child R_UTHUMB_S, origin xyz=0.0 0.023 -0.084 rpy=0.0 -0.0 0.0, axis 1.0 0.0 0.0, limit lower=-0.785398163397 upper=0.0 effort=100.0 velocity=6.80678
- added joint R_WRIST_R: type revolute, parent R_ELBOW_Y_S, child R_WRIST_R_S, origin xyz=0.0 2.77555756156e-16 -1.80411241502e-16 rpy=0.0 -0.0 0.0, axis 1.0 0.0 0.0, limit lower=-1.91986217719 upper=1.91986217719 effort=100.0 velocity=5.75958
- added joint R_WRIST_Y: type revolute, parent R_WRIST_R_S, child R_WRIST_Y_S, origin xyz=0.0 2.77555756156e-16 -1.80411241502e-16 rpy=0.0 -0.0 0.0, axis 0.0 0.0 1.0, limit lower=-2.61799387799 upper=2.61799387799 effort=100.0 velocity=3.66519
- added joint WAIST_P: type revolute, parent WAIST_Y_S, child WAIST_P_S, origin xyz=0.0 0.0 -1.11022302463e-16 rpy=0.0 -0.0 0.0, axis 0.0 1.0 0.0, limit lower=-0.523598775598 upper=1.0471975512 effort=100.0 velocity=8.90117
- added joint WAIST_R: type revolute, parent WAIST_P_S, child WAIST_R_S, origin xyz=0.0 0.0 -1.11022302463e-16 rpy=0.0 -0.0 0.0, axis 1.0 0.0 0.0, limit lower=-0.872664625997 upper=0.872664625997 effort=100.0 velocity=9.42477
- added joint WAIST_Y: type revolute, parent PELVIS_S, child WAIST_Y_S, origin xyz=0.0 0.0 0.192 rpy=0.0 -0.0 0.0, axis 0.0 0.0 1.0, limit lower=-0.785398163397 upper=0.785398163397 effort=100.0 velocity=8.90117
- added joint dcamera_JOINT: type fixed, parent NECK_P_S, child dcamera, origin xyz=0.1 0.0 0.09 rpy=-2.09440867144 1.64830267294e-05 -1.57082487668
- added joint gsensor_JOINT: type fixed, parent PELVIS_S, child gsensor, origin xyz=0.0 0.0 0.0 rpy=0.0 -0.0 0.0
- added joint gyrometer_JOINT: type fixed, parent PELVIS_S, child gyrometer, origin xyz=0.0 0.0 0.0 rpy=0.0 -0.0 0.0
- added joint l_ankle_joint: type fixed, parent L_ANKLE_P_S, child l_ankle, origin xyz=0 0 0 rpy=0 0 0
- added joint l_wrist_joint: type fixed, parent L_WRIST_Y_S, child l_wrist, origin xyz=0 0 0 rpy=0 0 0
- added joint lcamera_JOINT: type fixed, parent NECK_P_S, child lcamera, origin xyz=0.1 0.03 0.09 rpy=-2.09440867144 1.64830267294e-05 -1.57082487668
- added joint lfsensor_JOINT: type fixed, parent L_ANKLE_P_S, child lfsensor, origin xyz=0.0 0.0 0.0 rpy=0.0 -0.0 0.0
- added joint lhsensor_JOINT: type fixed, parent L_WRIST_Y_S, child lhsensor, origin xyz=0.0 0.0 0.0 rpy=0.0 -0.0 0.0
- added joint r_ankle_joint: type fixed, parent R_ANKLE_P_S, child r_ankle, origin xyz=0 0 0 rpy=0 0 0
- added joint r_wrist_joint: type fixed, parent R_WRIST_Y_S, child r_wrist, origin xyz=0 0 0 rpy=0 0 0
- added joint ranger_JOINT: type fixed, parent NECK_P_S, child ranger, origin xyz=0.1 0.0 0.0 rpy=1.90331089466e-05 0.523612344569 -1.9033108947e-05
- added joint rcamera_JOINT: type fixed, parent NECK_P_S, child rcamera, origin xyz=0.1 -0.03 0.09 rpy=-2.09440867144 1.64830267294e-05 -1.57082487668
- added joint rfsensor_JOINT: type fixed, parent R_ANKLE_P_S, child rfsensor, origin xyz=0.0 0.0 0.0 rpy=0.0 -0.0 0.0
- added joint rhsensor_JOINT: type fixed, parent R_WRIST_Y_S, child rhsensor, origin xyz=0.0 0.0 0.0 rpy=0.0 -0.0 0.0
- added joint waist: type fixed, parent base_link, child PELVIS_S, origin xyz=0 0 0 rpy=0 0 0
