Commit message: almost robot ealking with open loop is-mpc

File: g1_description/g1_29dof_lock_waist_with_hand_rev_1_0.urdf (robot description, URDF)
Before this commit: robot g1_29dof_lock_waist_with_hand_rev_1_0, 53 links, 52 joints
Links:
- added link left_foot_link, mass 0.00001; collision sphere radius=0.005; collision sphere radius=0.005
- added link right_foot_link, mass 0.00001; collision sphere radius=0.005; collision sphere radius=0.005
- link left_ankle_roll_link: geometry visual mesh filename=meshes/left_ankle_roll_link.STL
- link right_ankle_roll_link: geometry visual mesh filename=meshes/right_ankle_roll_link.STL
Joints:
- added joint left_foot_joint: type fixed, parent left_ankle_roll_link, child left_foot_link, origin xyz=0.035 0 -0.03 rpy=0 0 0, axis 1 0 0, limit lower=-0.2618 upper=0.2618 effort=35 velocity=30
- added joint right_foot_joint: type fixed, parent right_ankle_roll_link, child right_foot_link, origin xyz=0.035 0 -0.03 rpy=0 0 0, axis 1 0 0, limit lower=-0.2618 upper=0.2618 effort=35 velocity=30
