Commit message: final code for experiments

File: robot/g1/g1_description/g1_no_foot_link.urdf (robot description, URDF)
Before this commit: robot g1_29dof_lock_waist_with_hand_rev_1_0, 55 links, 54 joints
Links:
- removed link left_foot_link
- removed link right_foot_link
- link left_ankle_roll_link: geometry collision sphere radius=0.005; collision sphere radius=0.005
- link right_ankle_roll_link: geometry collision sphere radius=0.005; collision sphere radius=0.005
Joints:
- removed joint left_foot_joint
- removed joint right_foot_joint

File: robot/g1/g1_description/g1_norm_hand.urdf (robot description, URDF)
Before this commit: robot unitreeg1, 41 links, 40 joints
Links:
- added link waist_support_link, mass 0.001; collision mesh filename=meshes/waist_support_link.STL; visual mesh filename=meshes/waist_support_link.STL
- link torso_link: mass 6.78 -> 8.562; geometry collision mesh filename=meshes/torso_link.STL; visual mesh filename=meshes/torso_link.STL
- link waist_roll_link: mass 0.086 -> 0.047; geometry visual mesh filename=meshes/waist_roll_link.STL
- link waist_yaw_link: mass 0.214 -> 0.244; geometry visual mesh filename=meshes/waist_yaw_link.STL
Joints:
- added joint waist_support_joint: type fixed, parent torso_link, child waist_support_link, origin xyz=0.0039635 0 -0.054 rpy=0 0 0
- joint d435_joint: origin xyz=0.0576235 0.01753 0.42987 rpy=0 0.8307767239493009 0 -> xyz=0.0576235 0.01753 0.41987 rpy=0 0.8307767239493009 0
- joint head_joint: origin xyz=0.0039635 0 -0.044 rpy=0 0 0 -> xyz=0.0039635 0 -0.054 rpy=0 0 0
- joint imu_in_torso_joint: origin xyz=-0.03959 -0.00224 0.14792 rpy=0 0 0 -> xyz=-0.03959 -0.00224 0.13792 rpy=0 0 0
- joint left_hip_roll_joint: limit lower=-0.5236 upper=2.9671 effort=139 velocity=20 -> lower=-0.5236 upper=2.9671 effort=88 velocity=32
- joint left_shoulder_pitch_joint: origin xyz=0.0039563 0.10022 0.24778 rpy=0.27931 5.4949E-05 -0.00019159 -> xyz=0.0039563 0.10022 0.23778 rpy=0.27931 5.4949E-05 -0.00019159
- joint logo_joint: origin xyz=0.0039635 0 -0.044 rpy=0 0 0 -> xyz=0.0039635 0 -0.054 rpy=0 0 0
- joint mid360_joint: origin xyz=0.0002835 0.00003 0.41618 rpy=0 0.04014257279586953 0 -> xyz=0.0002835 0.00003 0.40618 rpy=0 0.04014257279586953 0
- joint right_hip_roll_joint: limit lower=-2.9671 upper=0.5236 effort=139 velocity=20 -> lower=-2.9671 upper=0.5236 effort=88 velocity=32
- joint right_shoulder_pitch_joint: origin xyz=0.0039563 -0.10021 0.24778 rpy=-0.27931 5.4949E-05 0.00019159 -> xyz=0.0039563 -0.10021 0.23778 rpy=-0.27931 5.4949E-05 0.00019159
- joint waist_pitch_joint: origin xyz=0 0 0 rpy=0 0 0 -> xyz=0 0 0.019 rpy=0 0 0
- joint waist_roll_joint: origin xyz=-0.0039635 0 0.044 rpy=0 0 0 -> xyz=-0.0039635 0 0.035 rpy=0 0 0

File: robot/g1/g1_description/g1_rev_hand.urdf (robot description, URDF)
Before this commit: robot g1_29dof_lock_waist_rev_1_0, 39 links, 38 joints
Links:
- removed link left_rubber_hand
- removed link right_rubber_hand
- added link left_foot_link, mass 0.00001; collision sphere radius=0.005; collision sphere radius=0.005
- added link left_hand_index_0_link, mass 0.05885070; collision mesh filename=meshes/left_hand_index_0_link.STL; visual mesh filename=meshes/left_hand_index_0_link.STL
- added link left_hand_index_1_link, mass 0.02030626; collision mesh filename=meshes/left_hand_index_1_link.STL; visual mesh filename=meshes/left_hand_index_1_link.STL
- added link left_hand_middle_0_link, mass 0.05885070; collision mesh filename=meshes/left_hand_middle_0_link.STL; visual mesh filename=meshes/left_hand_middle_0_link.STL
- added link left_hand_middle_1_link, mass 0.02030626; collision mesh filename=meshes/left_hand_middle_1_link.STL; visual mesh filename=meshes/left_hand_middle_1_link.STL
- added link left_hand_palm_link, mass 0.37283854; collision mesh filename=meshes/left_hand_palm_link.STL; visual mesh filename=meshes/left_hand_palm_link.STL
- added link left_hand_thumb_0_link, mass 0.08623657; collision mesh filename=meshes/left_hand_thumb_0_link.STL; visual mesh filename=meshes/left_hand_thumb_0_link.STL
- added link left_hand_thumb_1_link, mass 0.05885070; collision box size=0.02 0.03 0.02; visual mesh filename=meshes/left_hand_thumb_1_link.STL
- added link left_hand_thumb_2_link, mass 0.02030626; collision mesh filename=meshes/left_hand_thumb_2_link.STL; visual mesh filename=meshes/left_hand_thumb_2_link.STL
- added link right_foot_link, mass 0.00001; collision sphere radius=0.005; collision sphere radius=0.005
- added link right_hand_index_0_link, mass 0.05885070; collision mesh filename=meshes/right_hand_index_0_link.STL; visual mesh filename=meshes/right_hand_index_0_link.STL
- added link right_hand_index_1_link, mass 0.02030626; collision mesh filename=meshes/right_hand_index_1_link.STL; visual mesh filename=meshes/right_hand_index_1_link.STL
- added link right_hand_middle_0_link, mass 0.05885070; collision mesh filename=meshes/right_hand_middle_0_link.STL; visual mesh filename=meshes/right_hand_middle_0_link.STL
- added link right_hand_middle_1_link, mass 0.02030626; collision mesh filename=meshes/right_hand_middle_1_link.STL; visual mesh filename=meshes/right_hand_middle_1_link.STL
- added link right_hand_palm_link, mass 0.37283854; collision mesh filename=meshes/right_hand_palm_link.STL; visual mesh filename=meshes/right_hand_palm_link.STL
- added link right_hand_thumb_0_link, mass 0.08623657; collision mesh filename=meshes/right_hand_thumb_0_link.STL; visual mesh filename=meshes/right_hand_thumb_0_link.STL
- added link right_hand_thumb_1_link, mass 0.05885070; collision box size=0.02 0.03 0.02; visual mesh filename=meshes/right_hand_thumb_1_link.STL
- added link right_hand_thumb_2_link, mass 0.02030626; collision mesh filename=meshes/right_hand_thumb_2_link.STL; visual mesh filename=meshes/right_hand_thumb_2_link.STL
- link left_ankle_roll_link: geometry visual mesh filename=meshes/left_ankle_roll_link.STL
- link right_ankle_roll_link: geometry visual mesh filename=meshes/right_ankle_roll_link.STL
Joints:
- added joint left_foot_joint: type fixed, parent left_ankle_roll_link, child left_foot_link, origin xyz=0.035 0 -0.03 rpy=0 0 0, axis 1 0 0
- added joint left_hand_index_0_joint: type fixed, parent left_hand_palm_link, child left_hand_index_0_link, origin xyz=0.0777 0.0016 0.0285 rpy=0 0 0, axis 0 0 1, limit lower=-1.57079632 upper=0 effort=1.4 velocity=12
- added joint left_hand_index_1_joint: type fixed, parent left_hand_index_0_link, child left_hand_index_1_link, origin xyz=0.0458 0 0 rpy=0 0 0, axis 0 0 1, limit lower=-1.74532925 upper=0 effort=1.4 velocity=12
- added joint left_hand_middle_0_joint: type fixed, parent left_hand_palm_link, child left_hand_middle_0_link, origin xyz=0.0777 0.0016 -0.0285 rpy=0 0 0, axis 0 0 1, limit lower=-1.57079632 upper=0 effort=1.4 velocity=12
- added joint left_hand_middle_1_joint: type fixed, parent left_hand_middle_0_link, child left_hand_middle_1_link, origin xyz=0.0458 0 0 rpy=0 0 0, axis 0 0 1, limit lower=-1.74532925 upper=0 effort=1.4 velocity=12
- added joint left_hand_thumb_0_joint: type fixed, parent left_hand_palm_link, child left_hand_thumb_0_link, origin xyz=0.0255 0 0 rpy=0 0 0, axis 0 1 0, limit lower=-1.04719755 upper=1.04719755 effort=2.45 velocity=3.14
- added joint left_hand_thumb_1_joint: type fixed, parent left_hand_thumb_0_link, child left_hand_thumb_1_link, origin xyz=-0.0025 -0.0193 0 rpy=0 0 0, axis 0 0 1, limit lower=-0.61086523 upper=1.04719755 effort=1.4 velocity=12
- added joint left_hand_thumb_2_joint: type fixed, parent left_hand_thumb_1_link, child left_hand_thumb_2_link, origin xyz=0 -0.0458 0 rpy=0 0 0, axis 0 0 1, limit lower=0 upper=1.74532925 effort=1.4 velocity=12
- added joint right_foot_joint: type fixed, parent right_ankle_roll_link, child right_foot_link, origin xyz=0.035 0 -0.03 rpy=0 0 0, axis 1 0 0
- added joint right_hand_index_0_joint: type fixed, parent right_hand_palm_link, child right_hand_index_0_link, origin xyz=0.0777 -0.0016 0.0285 rpy=0 0 0, axis 0 0 1, limit lower=0 upper=1.57079632 effort=1.4 velocity=12
- added joint right_hand_index_1_joint: type fixed, parent right_hand_index_0_link, child right_hand_index_1_link, origin xyz=0.0458 0 0 rpy=0 0 0, axis 0 0 1, limit lower=0 upper=1.74532925 effort=1.4 velocity=12
- added joint right_hand_middle_0_joint: type fixed, parent right_hand_palm_link, child right_hand_middle_0_link, origin xyz=0.0777 -0.0016 -0.0285 rpy=0 0 0, axis 0 0 1, limit lower=0 upper=1.57079632 effort=1.4 velocity=12
- added joint right_hand_middle_1_joint: type fixed, parent right_hand_middle_0_link, child right_hand_middle_1_link, origin xyz=0.0458 0 0 rpy=0 0 0, axis 0 0 1, limit lower=0 upper=1.74532925 effort=1.4 velocity=12
- added joint right_hand_thumb_0_joint: type fixed, parent right_hand_palm_link, child right_hand_thumb_0_link, origin xyz=0.0255 0 0 rpy=0 0 0, axis 0 1 0, limit lower=-1.04719755 upper=1.04719755 effort=2.45 velocity=3.14
- added joint right_hand_thumb_1_joint: type fixed, parent right_hand_thumb_0_link, child right_hand_thumb_1_link, origin xyz=-0.0025 0.0193 0 rpy=0 0 0, axis 0 0 1, limit lower=-1.04719755 upper=0.61086523 effort=1.4 velocity=12
- added joint right_hand_thumb_2_joint: type fixed, parent right_hand_thumb_1_link, child right_hand_thumb_2_link, origin xyz=0 0.0458 0 rpy=0 0 0, axis 0 0 1, limit lower=-1.74532925 upper=0 effort=1.4 velocity=12
- joint left_hand_palm_joint: child left_rubber_hand -> left_hand_palm_link
- joint right_hand_palm_joint: child right_rubber_hand -> right_hand_palm_link
