Commit message: commit

File: robot/g1/g1_description/g1_rev_hand.urdf (robot description, URDF)
Before this commit: robot g1_rev_hand, 55 links, 54 joints
Joints:
- joint left_hand_index_0_joint: type fixed -> revolute
- joint left_hand_index_1_joint: type fixed -> revolute
- joint left_hand_middle_0_joint: type fixed -> revolute
- joint left_hand_middle_1_joint: type fixed -> revolute
- joint left_hand_thumb_0_joint: type fixed -> revolute
- joint left_hand_thumb_1_joint: type fixed -> revolute
- joint left_hand_thumb_2_joint: type fixed -> revolute
- joint right_hand_index_0_joint: type fixed -> revolute
- joint right_hand_index_1_joint: type fixed -> revolute
- joint right_hand_middle_0_joint: type fixed -> revolute
- joint right_hand_middle_1_joint: type fixed -> revolute
- joint right_hand_thumb_0_joint: type fixed -> revolute
- joint right_hand_thumb_1_joint: type fixed -> revolute
- joint right_hand_thumb_2_joint: type fixed -> revolute
