Commit message: works on filter

File: robot/g1/g1_description/g1_29dof_rev_1_0.urdf (robot description, URDF)
Before this commit: robot g1_29dof_rev_1_0, 41 links, 40 joints
Joints:
- joint left_foot_joint: origin xyz=0.035 0 -0.03 rpy=0 0 0 -> xyz=0.035 0 -0.0373314 rpy=0 0 0
- joint right_foot_joint: origin xyz=0.035 0 -0.03 rpy=0 0 0 -> xyz=0.035 0 -0.0373314 rpy=0 0 0

Commit message: commit

File: robot/g1/g1_description/g1_29dof_rev_1_0.urdf (robot description, URDF)
Before this commit: robot g1_29dof_rev_1_0, 41 links, 40 joints
Joints:
- joint left_foot_joint: origin xyz=0.035 0 -0.0373314 rpy=0 0 0 -> xyz=0.035 0 -0.035 rpy=0 0 0
- joint right_foot_joint: origin xyz=0.035 0 -0.0373314 rpy=0 0 0 -> xyz=0.035 0 -0.035 rpy=0 0 0
