Commit message: update

File: robot/g1/g1_description/g1_29dof_with_hand_rev_1_0.urdf (robot description, URDF)
Before this commit: robot g1_29dof_rev_1_0, 41 links, 40 joints
Links:
- removed link left_rubber_hand
- removed link right_rubber_hand
- added link left_hand_index_0_link, mass 0.05885070; collision mesh filename=meshes/left_hand_index_0_link.STL; visual mesh filename=meshes/left_hand_index_0_link.STL
- added link left_hand_index_1_link, mass 0.02030626; collision mesh filename=meshes/left_hand_index_1_link.STL; visual mesh filename=meshes/left_hand_index_1_link.STL
- added link left_hand_middle_0_link, mass 0.05885070; collision mesh filename=meshes/left_hand_middle_0_link.STL; visual mesh filename=meshes/left_hand_middle_0_link.STL
- added link left_hand_middle_1_link, mass 0.02030626; collision mesh filename=meshes/left_hand_middle_1_link.STL; visual mesh filename=meshes/left_hand_middle_1_link.STL
- added link left_hand_palm_link, mass 0.37283854; collision mesh filename=meshes/left_hand_palm_link.STL; visual mesh filename=meshes/left_hand_palm_link.STL
- added link left_hand_thumb_0_link, mass 0.08623657; collision mesh filename=meshes/left_hand_thumb_0_link.STL; visual mesh filename=meshes/left_hand_thumb_0_link.STL
- added link left_hand_thumb_1_link, mass 0.05885070; collision box size=0.02 0.03 0.02; visual mesh filename=meshes/left_hand_thumb_1_link.STL
- added link left_hand_thumb_2_link, mass 0.02030626; collision mesh filename=meshes/left_hand_thumb_2_link.STL; visual mesh filename=meshes/left_hand_thumb_2_link.STL
- added link right_hand_index_0_link, mass 0.05885070; collision mesh filename=meshes/right_hand_index_0_link.STL; visual mesh filename=meshes/right_hand_index_0_link.STL
- added link right_hand_index_1_link, mass 0.02030626; collision mesh filename=meshes/right_hand_index_1_link.STL; visual mesh filename=meshes/right_hand_index_1_link.STL
- added link right_hand_middle_0_link, mass 0.05885070; collision mesh filename=meshes/right_hand_middle_0_link.STL; visual mesh filename=meshes/right_hand_middle_0_link.STL
- added link right_hand_middle_1_link, mass 0.02030626; collision mesh filename=meshes/right_hand_middle_1_link.STL; visual mesh filename=meshes/right_hand_middle_1_link.STL
- added link right_hand_palm_link, mass 0.37283854; collision mesh filename=meshes/right_hand_palm_link.STL; visual mesh filename=meshes/right_hand_palm_link.STL
- added link right_hand_thumb_0_link, mass 0.08623657; collision mesh filename=meshes/right_hand_thumb_0_link.STL; visual mesh filename=meshes/right_hand_thumb_0_link.STL
- added link right_hand_thumb_1_link, mass 0.05885070; collision box size=0.02 0.03 0.02; visual mesh filename=meshes/right_hand_thumb_1_link.STL
- added link right_hand_thumb_2_link, mass 0.02030626; collision mesh filename=meshes/right_hand_thumb_2_link.STL; visual mesh filename=meshes/right_hand_thumb_2_link.STL
Joints:
- added joint left_hand_index_0_joint: type fixed, parent left_hand_palm_link, child left_hand_index_0_link, origin xyz=0.0777 0.0016 0.0285 rpy=0 0 0, axis 0 0 1, limit lower=-1.57079632 upper=0 effort=1.4 velocity=12
- added joint left_hand_index_1_joint: type fixed, parent left_hand_index_0_link, child left_hand_index_1_link, origin xyz=0.0458 0 0 rpy=0 0 0, axis 0 0 1, limit lower=-1.74532925 upper=0 effort=1.4 velocity=12
- added joint left_hand_middle_0_joint: type fixed, parent left_hand_palm_link, child left_hand_middle_0_link, origin xyz=0.0777 0.0016 -0.0285 rpy=0 0 0, axis 0 0 1, limit lower=-1.57079632 upper=0 effort=1.4 velocity=12
- added joint left_hand_middle_1_joint: type fixed, parent left_hand_middle_0_link, child left_hand_middle_1_link, origin xyz=0.0458 0 0 rpy=0 0 0, axis 0 0 1, limit lower=-1.74532925 upper=0 effort=1.4 velocity=12
- added joint left_hand_thumb_0_joint: type fixed, parent left_hand_palm_link, child left_hand_thumb_0_link, origin xyz=0.0255 0 0 rpy=0 0 0, axis 0 1 0, limit lower=-1.04719755 upper=1.04719755 effort=2.45 velocity=3.14
- added joint left_hand_thumb_1_joint: type fixed, parent left_hand_thumb_0_link, child left_hand_thumb_1_link, origin xyz=-0.0025 -0.0193 0 rpy=0 0 0, axis 0 0 1, limit lower=-0.61086523 upper=1.04719755 effort=1.4 velocity=12
- added joint left_hand_thumb_2_joint: type fixed, parent left_hand_thumb_1_link, child left_hand_thumb_2_link, origin xyz=0 -0.0458 0 rpy=0 0 0, axis 0 0 1, limit lower=0 upper=1.74532925 effort=1.4 velocity=12
- added joint right_hand_index_0_joint: type fixed, parent right_hand_palm_link, child right_hand_index_0_link, origin xyz=0.0777 -0.0016 0.0285 rpy=0 0 0, axis 0 0 1, limit lower=0 upper=1.57079632 effort=1.4 velocity=12
- added joint right_hand_index_1_joint: type fixed, parent right_hand_index_0_link, child right_hand_index_1_link, origin xyz=0.0458 0 0 rpy=0 0 0, axis 0 0 1, limit lower=0 upper=1.74532925 effort=1.4 velocity=12
- added joint right_hand_middle_0_joint: type fixed, parent right_hand_palm_link, child right_hand_middle_0_link, origin xyz=0.0777 -0.0016 -0.0285 rpy=0 0 0, axis 0 0 1, limit lower=0 upper=1.57079632 effort=1.4 velocity=12
- added joint right_hand_middle_1_joint: type fixed, parent right_hand_middle_0_link, child right_hand_middle_1_link, origin xyz=0.0458 0 0 rpy=0 0 0, axis 0 0 1, limit lower=0 upper=1.74532925 effort=1.4 velocity=12
- added joint right_hand_thumb_0_joint: type fixed, parent right_hand_palm_link, child right_hand_thumb_0_link, origin xyz=0.0255 0 0 rpy=0 0 0, axis 0 1 0, limit lower=-1.04719755 upper=1.04719755 effort=2.45 velocity=3.14
- added joint right_hand_thumb_1_joint: type fixed, parent right_hand_thumb_0_link, child right_hand_thumb_1_link, origin xyz=-0.0025 0.0193 0 rpy=0 0 0, axis 0 0 1, limit lower=-1.04719755 upper=0.61086523 effort=1.4 velocity=12
- added joint right_hand_thumb_2_joint: type fixed, parent right_hand_thumb_1_link, child right_hand_thumb_2_link, origin xyz=0 0.0458 0 rpy=0 0 0, axis 0 0 1, limit lower=-1.74532925 upper=0 effort=1.4 velocity=12
- joint left_foot_joint: origin xyz=0.035 0 -0.030 rpy=0 0 0 -> xyz=0.035 0 -0.0338 rpy=0 0 0
- joint left_hand_palm_joint: child left_rubber_hand -> left_hand_palm_link
- joint mid360_joint: origin xyz=0.0002835 0.00003 0.41618 rpy=0 0.04014257279586953 0 -> xyz=0.0002835 0.00003 0.428434 rpy=3.141592653589793 0.05112069379091391 0
- joint right_foot_joint: origin xyz=0.035 0 -0.030 rpy=0 0 0 -> xyz=0.035 0 -0.0338 rpy=0 0 0
- joint right_hand_palm_joint: child right_rubber_hand -> right_hand_palm_link
