Commit message: removed diligentkio, cleanup

File: robot/g1/g1_description/g1_29dof_lock_waist_with_hand_rev_1_0.urdf (robot description, URDF)
Before this commit: robot g1_rev_hand, 53 links, 52 joints
Links:
- added link left_foot_link, mass 0.00001; collision sphere radius=0.005; collision sphere radius=0.005
- added link right_foot_link, mass 0.00001; collision sphere radius=0.005; collision sphere radius=0.005
- link left_ankle_roll_link: geometry visual mesh filename=meshes/left_ankle_roll_link.STL
- link right_ankle_roll_link: geometry visual mesh filename=meshes/right_ankle_roll_link.STL
Joints:
- added joint left_foot_joint: type fixed, parent left_ankle_roll_link, child left_foot_link, origin xyz=0.035 0 -0.0338 rpy=0 0 0, axis 1 0 0
- added joint right_foot_joint: type fixed, parent right_ankle_roll_link, child right_foot_link, origin xyz=0.035 0 -0.0338 rpy=0 0 0, axis 1 0 0
- joint left_hand_index_0_joint: type fixed -> revolute
- joint left_hand_index_1_joint: type fixed -> revolute
- joint left_hand_middle_0_joint: type fixed -> revolute
- joint left_hand_middle_1_joint: type fixed -> revolute
- joint left_hand_thumb_0_joint: type fixed -> revolute
- joint left_hand_thumb_1_joint: type fixed -> revolute
- joint left_hand_thumb_2_joint: type fixed -> revolute
- joint mid360_joint: origin xyz=0.0002835 0.00003 0.41618 rpy=0 0.04014257279586953 0 -> xyz=0.0002835 0.00003 0.428434 rpy=3.141592653589793 0.05112069379091391 0
- joint right_hand_index_0_joint: type fixed -> revolute
- joint right_hand_index_1_joint: type fixed -> revolute
- joint right_hand_middle_0_joint: type fixed -> revolute
- joint right_hand_middle_1_joint: type fixed -> revolute
- joint right_hand_thumb_0_joint: type fixed -> revolute
- joint right_hand_thumb_1_joint: type fixed -> revolute
- joint right_hand_thumb_2_joint: type fixed -> revolute

Commit message: don't use not working

File: robot/g1/g1_description/g1_29dof_lock_waist_with_hand_rev_1_0.urdf (robot description, URDF)
Before this commit: robot g1_29dof_lock_waist_with_hand_rev_1_0, 55 links, 54 joints
Joints:
- joint left_hand_index_0_joint: type revolute -> fixed
- joint left_hand_index_1_joint: type revolute -> fixed
- joint left_hand_middle_0_joint: type revolute -> fixed
- joint left_hand_middle_1_joint: type revolute -> fixed
- joint left_hand_thumb_0_joint: type revolute -> fixed
- joint left_hand_thumb_1_joint: type revolute -> fixed
- joint left_hand_thumb_2_joint: type revolute -> fixed
- joint right_hand_index_0_joint: type revolute -> fixed
- joint right_hand_index_1_joint: type revolute -> fixed
- joint right_hand_middle_0_joint: type revolute -> fixed
- joint right_hand_middle_1_joint: type revolute -> fixed
- joint right_hand_thumb_0_joint: type revolute -> fixed
- joint right_hand_thumb_1_joint: type revolute -> fixed
- joint right_hand_thumb_2_joint: type revolute -> fixed
