Commit message: first iteration, gives seg fault, merge main

File: robot/gene01/gene01_description/gene01.urdf (robot description, URDF)
Before this commit: robot gene01, 91 links, 90 joints
Joints:
- joint l_sole_fixed_joint: origin xyz=-0.015 0 -0.036 rpy=0 0 0 -> xyz=0.045 0 -0.036 rpy=0 0 0
- joint l_wrist_pitch: type revolute -> fixed
- joint l_wrist_roll: type revolute -> fixed
- joint l_wrist_yaw: type revolute -> fixed
- joint r_sole_fixed_joint: origin xyz=-0.015 0 -0.036 rpy=0 0 0 -> xyz=0.045 0 -0.036 rpy=0 0 0
- joint r_wrist_pitch: type revolute -> fixed
- joint r_wrist_roll: type revolute -> fixed
- joint r_wrist_yaw: type revolute -> fixed
- joint torso_roll: type revolute -> fixed
